File: e155-DS1722-board.kicad_pcb (KiCad board)
At the start: 2 copper layers, 0 parts

Commit message: Initial PCB layout and routing
Parts:
- added D1: LED, LED_SMD:LED_0805_2012Metric, F.Cu at (118.5, 84.2)
- added D2: LED, LED_SMD:LED_0805_2012Metric, F.Cu at (110.0, 75.3)
- added D3: LED, LED_SMD:LED_0805_2012Metric, F.Cu at (116.2, 75.4)
- added D4: LED, LED_SMD:LED_0805_2012Metric, F.Cu at (115.1, 91.2)
- added D5: LED, LED_SMD:LED_0805_2012Metric, F.Cu at (110.5, 91.2)
- added J1: Conn_01x08, Connector_PinHeader_2.54mm:PinHeader_1x08_P2.54mm_Vertical, F.Cu at (100.3, 74.4)
- added J2: Conn_01x08, Connector_PinHeader_2.54mm:PinHeader_1x08_P2.54mm_Vertical, F.Cu at (123.2, 74.4)
- added R1: 1k, Resistor_SMD:R_0805_2012Metric, F.Cu at (118.5, 80.4)
- added R2: 1k, Resistor_SMD:R_0805_2012Metric, F.Cu at (110.0, 71.5)
- added R3: 1k, Resistor_SMD:R_0805_2012Metric, F.Cu at (116.2, 71.5)
- added R4: 1k, Resistor_SMD:R_0805_2012Metric, F.Cu at (115.1, 95.0)
- added R5: 1k, Resistor_SMD:R_0805_2012Metric, F.Cu at (110.5, 95.0)
- added U1: ~, Package_SO:SOIC-8_3.9x4.9mm_P1.27mm, F.Cu at (112.4, 82.2)
Routing:
- net /+3.3V: track 0.00 -> 42.9 mm, vias 0 -> 1
- net /CS: track 0.00 -> 36.4 mm
- net /SCK: track 0.00 -> 21.1 mm
- net /MOSI: track 0.00 -> 20.3 mm
- net /MISO: track 0.00 -> 17.5 mm, vias 0 -> 2
- net Net-(D3-K): track 0.00 -> 2.06 mm
- net Net-(D5-K): track 0.00 -> 1.94 mm
- net Net-(D2-K): track 0.00 -> 1.94 mm
- net Net-(D1-K): track 0.00 -> 1.94 mm
- net Net-(D4-K): track 0.00 -> 1.91 mm
- added copper zone on F.Cu, net GND
Other:
- board outline added: 27.9 x 28.6 mm
